File: power.kicad_sch (KiCad schematic)
At the start: 49 parts, among them J201 -, J202 -, J203 Barrel_Jack_MountingPin, Q201 AOD4185, U101 74HC04, U102 74HC08, U103 74HC32, U201 MP9942GJ

Commit message: Add pulldowns and make all pulldowns larger
Parts:
- J201: footprint _my:PinHeader_1x02_P2.54mm_Vertical_min -> _my:PinHeader_1x04_P2.54mm_Vertical_min_1
- J202: footprint _my:PinHeader_01x03_P2.5mm_Vertical_min -> _my:PinHeader_01x02_P5mm_Vertical_min
- J203: footprint _my:BarrelJack_2.1mm -> _my:BarrelJack_2.1mm_SMD
Changed lines of the file:
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@@
       (effects (font (size 1.27 1.27)))
     )
-    (property "Footprint" "_my:BarrelJack_2.1mm" (at 36.83 41.656 0)
+    (property "Footprint" "_my:BarrelJack_2.1mm_SMD" (at 36.83 41.656 0)
       (effects (font (size 1.27 1.27)) hide)
     )
@@
       (effects (font (size 1.27 1.27)) (justify left))
     )
-    (property "Footprint" "_my:PinHeader_01x03_P2.5mm_Vertical_min" (at 66.04 39.37 0)
+    (property "Footprint" "_my:PinHeader_01x02_P5mm_Vertical_min" (at 66.04 39.37 0)
       (effects (font (size 1.27 1.27)) hide)
     )
@@
       (effects (font (size 1.27 1.27)) (justify left))
     )
-    (property "Footprint" "_my:PinHeader_1x02_P2.54mm_Vertical_min" (at 66.04 30.48 0)
-      (effects (font (size 1.27 1.27)) hide)
-    )
+    (property "Footprint" "_my:PinHeader_1x04_P2.54mm_Vertical_min_1" (at 66.04 30.48 0)
+      (effects (font (size 1.27 1.27)) hide)
+    )
