File: power.kicad_sch (KiCad schematic)
At the start: 49 parts, among them J201 -, J202 -, J203 Barrel_Jack_MountingPin, Q201 AOD4185, U101 74HC04, U102 74HC08, U103 74HC32, U201 MP9942GJ

Commit message: Rev A2
Parts:
- J201: renamed from J203; footprint _my:BarrelJack_2.1mm -> _my:BarrelJack_2.1mm_SMD; LCSC Part # C194407 -> C2936010
- J202: footprint _my:PinHeader_01x03_P2.5mm_Vertical_min -> _my:PinHeader_01x02_P5mm_Vertical_min
- J203: renamed from J201; footprint _my:PinHeader_1x02_P2.54mm_Vertical_min -> _my:PinHeader_1x04_P2.54mm_Vertical_min_1
- JP203: renamed from JP202; footprint Jumper:SolderJumper-2_P1.3mm_Bridged2Bar_RoundedPad1.0x1.5mm -> _my:SolderJumper-2_P1.3mm_Bridged
- JP204: renamed from JP203; footprint Jumper:SolderJumper-2_P1.3mm_Bridged2Bar_RoundedPad1.0x1.5mm -> _my:SolderJumper-2_P1.3mm_Bridged
- renumbered C208 to C201, C209 to C202, C210 to C203, C211 to C204, C212 to C205, C213 to C206, C214 to C207, C215 to C208, C216 to C209, C217 to C210, C218 to C211, C201 to C212, C202 to C213, C203 to C214, C204 to C215, C205 to C216, C206 to C217, C207 to C218, JP204 to JP201, JP201 to JP202, R208 to R201, R201 to R202, R202 to R203, R207 to R204, R203 to R205, R204 to R206, R205 to R207, R206 to R208
Connections:
- net GND: now also J201.MP (MountPin), J203.2 (Pin_2)
- net v_conn: no longer J203.2 (Pin_2)
- no-connect marks 1 -> 0
Other:
- note removed: "Bulk Caps"
- moved on the sheet: C201, C202, C203, C204, C205, C206, C207, C208, C209, C210, C211, C212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

Commit message: update to RevB
Parts:
- removed C206, C207: -, Capacitor_SMD:C_1210_3225Metric_Pad1.33x2.70mm_HandSolder, symbol Device:C_Small
- removed C213: 10u VM 0805, Capacitor_SMD:C_0805_2012Metric, symbol Device:C_Small
- removed C218: 100n, _my:C_1005_(0402), symbol Device:C_Small
- removed JP204: Jumper_2, _my:SolderJumper-2_P1.3mm_Bridged, symbol Jumper:Jumper_2_Bridged
- removed Q201: AOD4185, Package_TO_SOT_SMD:TO-252-2, symbol _my:AOD4185
- removed R202, R205: 470k, _my:R_1005_(0402), symbol Device:R_Small
- removed R206, R207: 47k, _my:R_1005_(0402), symbol Device:R_Small
- removed R208: 5k76, _my:R_1005_(0402), symbol Device:R_Small
- removed U201: MP9942GJ, _my:TSOT23-8, symbol _my:MP9942GJ
- added C215: 56p, _my:C_1005_(0402), symbol Device:C_Small
- added JP204: Jumper_2_o, Jumper:SolderJumper-2_P1.3mm_Open_RoundedPad1.0x1.5mm, symbol Jumper:Jumper_2_Open
- added Q201: AO4407C, Package_SO:SOIC-8_3.9x4.9mm_P1.27mm, symbol Transistor_FET:IRF7404
- added R204: 9k1, _my:R_1005_(0402), symbol Device:R_Small
- added U201: TPS54302, Package_TO_SOT_SMD:SOT-23-6, symbol Regulator_Switching:TPS54302
- C201, C202: LCSC Part # C125975 -> C2972719; rohs_cert_or_in_datasheet y -> (none)
- C203, D201, D202, R201, U101, U102, U103: rohs_cert_or_in_datasheet y -> (none)
- C208: renamed from C212; rohs_cert_or_in_datasheet y -> (none)
- C209: renamed from C205; rohs_cert_or_in_datasheet y -> (none)
- C210: renamed from C204; rohs_cert_or_in_datasheet y -> (none)
- C211: renamed from C214; rohs_cert_or_in_datasheet y -> (none)
- C212: renamed from C215; rohs_cert_or_in_datasheet y -> (none)
- C213: renamed from C216; rohs_cert_or_in_datasheet y -> (none)
- C214: renamed from C217; rohs_cert_or_in_datasheet y -> (none)
- C216: renamed from C219; rohs_cert_or_in_datasheet y -> (none)
- C217: renamed from C220; rohs_cert_or_in_datasheet y -> (none)
- C218: renamed from C221; rohs_cert_or_in_datasheet y -> (none)
- C219: renamed from C222; rohs_cert_or_in_datasheet y -> (none)
- C220: renamed from C223; rohs_cert_or_in_datasheet y -> (none)
- C221: renamed from C224; rohs_cert_or_in_datasheet y -> (none)
- C222: renamed from C225; rohs_cert_or_in_datasheet y -> (none)
- J201: LCSC Part # C2936010 -> C319134; rohs_cert_or_in_datasheet n -> (none)
- L201: value 56uH -> 15uH; footprint _my:L_PSPMAA0805 -> 0_my:L_7.1x6.6_H3_SLO0630H; LCSC Part # C2962890 -> C182182; rohs_cert_or_in_datasheet y -> (none)
- R202: renamed from R204; rohs_cert_or_in_datasheet y -> (none)
- R203: value 20R -> 100k; LCSC Part # C138031 -> C60491; rohs_cert_or_in_datasheet y -> (none)
- renumbered C208 to C204, C209 to C205, C210 to C206, C211 to C207
Connections:
- net GND: now also JP204.1 (A), R204.2, U201.1 (GND)
- net VM: now also Q201.1 (S), Q201.2 (S), Q201.3 (S), U201.3 (VIN)
- net bst: now also C208.1, U201.6 (BOOT); no longer R203.1
- net en2: now also JP204.2 (B), U201.5 (EN)
- net fn: now also R203.2, C215.1, R204.1, U201.4 (FB)
- net gate: now also Q201.4 (G)
- net sw: now also U201.2 (SW)
- net v_conn: now also Q201.5 (D), Q201.6 (D), Q201.7 (D), Q201.8 (D)
- net vin: now also R203.1, C215.2
Other:
- note added: "Output Voltage accorting to formula (3) in the Data Sheet: >>> 0.596*((100050/9100)+1) 7.148725274725274"
- note removed: "9V: ~4k7 7V5: ~5k5 5k76: ~7V2"
- moved on the sheet: C204, C205, C206, C207, C208, C209, C210, C211, C212, C213, C214, D202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
