File: motor-shield.kicad_sch (KiCad schematic)
At the start: 67 parts, among them J101 MC 1,5/ 2-G-3,5, J102 -, J103 MC 1,5/ 2-G-3,5, J104 -, J105 STEMMA QT, J106 Conn_02x04_smd, J107 Conn_01x04_f, Q101 AO3400A, Q102 AO3400A, SW101 Switch, U101 74HC04, U102 74HC08, U103 74HC32, U104 DRV8874PWPR, U105 DRV8874PWPR, U106 LMV321

Commit message: Rev A2
Parts:
- added R103, R104: 47k, _my:R_1005_(0402), symbol Device:R_Small
- JP101, JP102, JP103, JP105, JP106, JP108, JP109, JP110, JP111, JP112, JP113, JP114, JP115, JP116, JP117: footprint Jumper:SolderJumper-3_P1.3mm_Bridged12_RoundedPad1.0x1.5mm -> _my:SolderJumper-3
- renumbered R103 to R105, R104 to R106, R107 to R109, R108 to R110, R109 to R111, R110 to R112, R111 to R113, R112 to R114, R113 to R115, R114 to R116
Connections:
- net GND: now also R103.2, R104.2
- net pwm_a: now also R103.1
- net pwm_b: now also R104.1
Other:
- moved on the sheet: R101, R102

Commit message: update to RevB
Parts:
- C101, C102, C103, C104, C105, C106, C107, C108, C109, C110, C112, C113, C114, C115, C215, Q101, Q102, R101, R102, R103, R104, R109, R110, R111, R112, R204, SW101, U101, U102, U103, U104, U105, U106: rohs_cert_or_in_datasheet y -> (none)
- D203: value 0603_LED_Red -> 0603_LED_Yellow; rohs_cert_or_in_datasheet y -> (none)
- J101, J103: LCSC Part # C880572 -> C409115; rohs_cert_or_in_datasheet n -> (none)
- J105: rohs_cert_or_in_datasheet obtainable -> (none)
- J106: rohs_cert_or_in_datasheet n -> (none)
- J107: LCSC Part # C2935975 -> C2685089; rohs_cert_or_in_datasheet n -> (none)
- R113, R114: LCSC Part # C137939 -> C321605; rohs_cert_or_in_datasheet y -> (none)
- R115: value 47k -> 9k1; LCSC Part # C163440 -> C25926; rohs_cert_or_in_datasheet y -> (none)
- R116: value 470k -> 100k; LCSC Part # C137865 -> C60491; rohs_cert_or_in_datasheet y -> (none)
